Commit message: add turtlebot3 files
add turtlebot3 files for tutorials
changed the gitignore file for /devel
initialize devel branch for each member to use

File: src/turtlebot3/turtlebot3_description/urdf/turtlebot3_burger.urdf.xacro (robot description, xacro)
@@ -140,3 +140,25 @@
     </inertial>
   </link>
+<joint name="sonar_front_joint" type="fixed">
+    <axis xyz="0 0 0" />
+    <origin rpy="0 0 0" xyz="0.5 0 0.25" />
+    <parent link="base_footprint"/>
+    <child link="base_sonar_front"/>
+</joint><link name="base_sonar_front">
+    <collision>
+      <origin xyz="0 0 0" rpy="0 0 0"/>
+      <geometry>
+        <box size="0.01 0.01 0.01"/>
+      </geometry>
+    </collision>    <visual>
+      <origin xyz="0 0 0" rpy="0 0 0"/>
+      <geometry>
+        <box size="0.01 0.01 0.01"/>
+      </geometry>
+    </visual>    <inertial>
+      <mass value="1e-5" />
+      <origin xyz="0 0 0" rpy="0 0 0"/>
+      <inertia ixx="1e-6" ixy="0" ixz="0" iyy="1e-6" iyz="0" izz="1e-6" />
+    </inertial>
+ </link>
 </robot>

Commit message: Cartobot with Ultrasonic sensor
added the ultrasonic sensor to the  turtlebot3 burger.

currently the code can been used for making a map with lidar scanning.

File: src/turtlebot3/turtlebot3_description/urdf/turtlebot3_burger.urdf.xacro (robot description, xacro)
@@ -15,5 +15,5 @@
         <mesh filename="package://turtlebot3_description/meshes/bases/burger_base.stl" scale="0.001 0.001 0.001"/>
       </geometry>
-      <material name="light_black"/>
+      <material name="light_grey"/>
     </visual>
     <collision>
@@ -124,5 +124,5 @@
         <mesh filename="package://turtlebot3_description/meshes/sensors/lds.stl" scale="0.001 0.001 0.001"/>
       </geometry>
-      <material name="dark"/>
+      <material name="light_grey"/>
     </visual>
     <collision>
@@ -141,24 +141,30 @@
   </link>
 <joint name="sonar_front_joint" type="fixed">
-    <axis xyz="0 0 0" />
-    <origin rpy="0 0 0" xyz="0.5 0 0.25" />
+    <axis xyz="0 1 0" />
+    <origin rpy="0 0 0" xyz="0.038 -0.022 0.06" />
     <parent link="base_footprint"/>
     <child link="base_sonar_front"/>
-</joint><link name="base_sonar_front">
+</joint>
+<link name="base_sonar_front">
     <collision>
       <origin xyz="0 0 0" rpy="0 0 0"/>
       <geometry>
-        <box size="0.01 0.01 0.01"/>
+        <box size="0.03 0.03 0.03"/>
       </geometry>
-    </collision>    <visual>
+    </collision>
+   <visual>
+      <origin xyz="0 0 0" rpy=" 1.5707 0 1.5707"/>
+      <geometry>
+       <mesh filename="package://turtlebot3_description/meshes/sensors/sonar.stl" scale="0.001 0.001 0.001"/>
+      </geometry>
+      <material name="blue"/>
+    </visual>
+   <inertial>
+      <mass value="0.005" />
       <origin xyz="0 0 0" rpy="0 0 0"/>
-      <geometry>
-        <box size="0.01 0.01 0.01"/>
-      </geometry>
-    </visual>    <inertial>
-      <mass value="1e-5" />
-      <origin xyz="0 0 0" rpy="0 0 0"/>
-      <inertia ixx="1e-6" ixy="0" ixz="0" iyy="1e-6" iyz="0" izz="1e-6" />
-    </inertial>
+      <inertia ixx="0.01" ixy="0.0" ixz="0.0"
+               iyy="0.01" iyz="0.0"
+               izz="0.01" />
+     </inertial>
  </link>
 </robot>
