Commit message: visualization of the ultrasonic sensor
- make a simulator for display working of the ultrasonic sensor.
- In the simulation, the sensor is capable of detecting thresholds,
ramps and angled planes (like an angled table leg of the gzaebo cafe
table model)

- created a readme file on how the execute the different parts of the
cartobot project.

File: src/turtlebot3/turtlebot3_description/urdf/turtlebot3_burger.gazebo.xacro (robot description, xacro)
@@ -124,3 +124,41 @@
     </sensor>
   </gazebo>
+<gazebo reference="base_sonar_front">
+   <sensor type="ray" name="TeraRanger">
+      <origin xyz="0 1 0"/>
+      <pose>0 -10.5 0 0 0 0</pose>
+      <visualize>true</visualize>
+      <update_rate>15</update_rate>
+      <ray>
+         <scan>
+            <horizontal>
+               <samples>10</samples>
+               <resolution>2</resolution>
+               <min_angle>-0.25</min_angle>
+               <max_angle>0.25</max_angle>
+            </horizontal>
+            <vertical>
+               <samples>10</samples>
+               <resolution>5</resolution>
+               <min_angle>-0.25</min_angle>
+               <max_angle>0</max_angle>
+            </vertical>
+         </scan>
+         <range>
+            <min>0.1</min>
+            <max>2</max>
+            <resolution>0.05</resolution>
+         </range>
+      </ray>
+      <plugin filename="libgazebo_ros_range.so" name="gazebo_ros_range">
+         <gaussianNoise>0.005</gaussianNoise>
+         <alwaysOn>true</alwaysOn>
+         <updateRate>5</updateRate>
+         <topicName>sonar</topicName>
+         <frameName>base_sonar_front</frameName>
+         <radiation>ultrasound</radiation>
+         <fov>0.25</fov>
+      </plugin>
+   </sensor>
+   </gazebo>
 </robot>

File: src/turtlebot3/turtlebot3_description/urdf/turtlebot3_burger.urdf.xacro (robot description, xacro)
@@ -140,17 +140,11 @@
     </inertial>
   </link>
-<joint name="sonar_front_joint" type="fixed">
+ <joint name="sonar_front_joint" type="fixed">
     <axis xyz="0 1 0" />
     <origin rpy="0 0 0" xyz="0.038 -0.022 0.06" />
     <parent link="base_footprint"/>
     <child link="base_sonar_front"/>
-</joint>
-<link name="base_sonar_front">
-    <collision>
-      <origin xyz="0 0 0" rpy="0 0 0"/>
-      <geometry>
-        <box size="0.03 0.03 0.03"/>
-      </geometry>
-    </collision>
+ </joint>
+ <link name="base_sonar_front">
    <visual>
       <origin xyz="0 0 0" rpy=" 1.5707 0 1.5707"/>
@@ -160,4 +154,10 @@
       <material name="blue"/>
     </visual>
+    <collision>
+      <origin xyz="0 0 0" rpy="0 0 0"/>
+      <geometry>
+        <box size="0.03 0.03 0.03"/>
+      </geometry>
+    </collision>
    <inertial>
       <mass value="0.005" />

Commit message: ultra sonic V1.2
- change properties of sonar sensor
- callback functie in world.launch

File: src/turtlebot3/turtlebot3_description/urdf/turtlebot3_burger.gazebo.xacro (robot description, xacro)
@@ -1,4 +1,4 @@
 <?xml version="1.0"?>
-<robot name="turtlebot3_burger_sim" xmlns:xacro="http://ros.org/wiki/xacro">
+  <robot name="turtlebot3_burger_sim" xmlns:xacro="http://ros.org/wiki/xacro">
   <xacro:arg name="laser_visual" default="false"/>
   <xacro:arg name="imu_visual"   default="false"/>
@@ -126,5 +126,4 @@
 <gazebo reference="base_sonar_front">
    <sensor type="ray" name="TeraRanger">
-      <origin xyz="0 1 0"/>
       <pose>0 -10.5 0 0 0 0</pose>
       <visualize>true</visualize>
@@ -156,7 +155,7 @@
          <updateRate>5</updateRate>
          <topicName>sonar</topicName>
-         <frameName>base_sonar_front</frameName>
+         <frameName>base_sonar</frameName>
          <radiation>ultrasound</radiation>
-         <fov>0.25</fov>
+         <fov>0.3</fov>
       </plugin>
    </sensor>

Commit message: ultra sonic sensor WORKING
successfully implemented the ultra sonic sensor for detecting
thresholds.
for detecting of objects is uses both the lidar and sonar

File: src/turtlebot3/turtlebot3_description/urdf/turtlebot3_burger.gazebo.xacro (robot description, xacro)
@@ -124,14 +124,14 @@
     </sensor>
   </gazebo>
-<gazebo reference="base_sonar_front">
+<gazebo reference="base_sonar">
    <sensor type="ray" name="TeraRanger">
       <pose>0 -10.5 0 0 0 0</pose>
       <visualize>true</visualize>
-      <update_rate>10</update_rate>
+      <update_rate>50</update_rate>
       <ray>
          <scan>
             <horizontal>
                <samples>10</samples>
-               <resolution>2</resolution>
+               <resolution>5</resolution>
                <min_angle>-0.25</min_angle>
                <max_angle>0.25</max_angle>
@@ -140,12 +140,12 @@
                <samples>10</samples>
                <resolution>5</resolution>
-               <min_angle>-0.25</min_angle>
-               <max_angle>-0.05</max_angle>
+               <min_angle>-0.2</min_angle>
+               <max_angle>0</max_angle>
             </vertical>
          </scan>
          <range>
             <min>0.05</min>
-            <max>3</max>
-            <resolution>1</resolution>
+            <max>2</max>
+            <resolution>1.5</resolution>
          </range>
       </ray>
@@ -153,5 +153,5 @@
          <gaussianNoise>0.005</gaussianNoise>
          <alwaysOn>true</alwaysOn>
-         <updateRate>5</updateRate>
+         <updateRate>50</updateRate>
          <topicName>sonar</topicName>
          <frameName>base_sonar</frameName>

File: src/turtlebot3/turtlebot3_description/urdf/turtlebot3_burger.urdf.xacro (robot description, xacro)
@@ -140,11 +140,11 @@
     </inertial>
   </link>
- <joint name="sonar_front_joint" type="fixed">
+ <joint name="sonar_joint" type="fixed">
     <axis xyz="0 1 0" />
     <origin rpy="0 0 0" xyz="0.038 -0.022 0.06" />
     <parent link="base_footprint"/>
-    <child link="base_sonar_front"/>
+    <child link="base_sonar"/>
  </joint>
- <link name="base_sonar_front">
+ <link name="base_sonar">
    <visual>
       <origin xyz="0 0 0" rpy=" 1.5707 0 1.5707"/>
